Commit message: feat: animated iceberg

File: wamv_stonefish/scenarios/iceberg.scn.xacro (robot description, xacro)
@@ -11,5 +11,5 @@
     <xacro:include filename="$(find wamv_stonefish)/description/materials.scn.xacro"/>
     <xacro:include filename="$(find wamv_stonefish)/scenarios/ocean.scn.xacro"/>
-    <dynamic name="iceberg" type="model">
+    <!-- <static name="iceberg" type="model">
         <physical>
             <mesh filename="iceberg_01.obj" scale="1.0" convex="false"/>
@@ -22,6 +22,24 @@
         <material name="Ice"/>
         <look name="ice"/>
-        <!-- <mass value="500"/> -->
+        <cg xyz=" 0.0 0 0.0" rpy="0.0 0.0 0.0"/>
         <world_transform xyz="100.0 100.0 0.0" rpy="3.1415926 0.0 0.0"/>
-    </dynamic>
+    </static> -->
+    <animated name="AnimMesh" type="model" collisions="true">
+        <physical>
+            <mesh filename="iceberg_01.obj" scale="0.5" convex="false"/>
+            <origin xyz="0.0 0.0 0.0" rpy="0.0 0.0 0.0"/>
+        </physical>
+        <visual>
+            <mesh filename="iceberg_01.obj" scale="0.5"/>
+            <origin xyz="0.0 0.0 .0" rpy="0.0 0.0 0.0"/>
+        </visual>
+        <material name="Ice"/>
+        <look name="ice"/>
+        <world_transform xyz="100.0 100.0 0.0" rpy="3.1415926 0.0 0.0"/>
+        <trajectory type="spline" playback="boomerang">
+            <keypoint time="0.0" xyz="0.0 60.0 0.0" rpy="3.1415926 0.0 0.0"/>
+            <keypoint time="10.0" xyz="10.0 60.0 0.0" rpy="3.1415926 0.0 0"/>
+            <keypoint time="40.0" xyz="10.0 60.0 0.0" rpy="3.1415926 0.0 0.0"/>
+        </trajectory>
+    </animated>
 </scenario>
