Commit message: feat:added the engine

File: wamv_stonefish/description/wamv.scn.xacro (robot description, xacro)
@@ -13,5 +13,5 @@
         <robot name="${robot_name}" fixed="false" self_collisions="false">
             <base_link name="Vehicle" type="compound" physics="submerged">
-                <external_part name="Hull" type="model" physics="submerged" buoyant="true">
+                <external_part name="base" type="model" physics="submerged" buoyant="true">
                     <physical>
                         <mesh filename="wamv_base.obj" scale="0.0045"/>
@@ -25,16 +25,37 @@
                     <look name="yellow"/>
                     <mass value="50"/>
-                    <!-- <inertia xyz="1.0 1.0 1.0"/> -->
                     <compound_transform rpy="0.0 0.0 0.0" xyz="0.0 0.0 0.0"/>
                     <cg xyz=" 0.0 0 1.0" rpy="0.0 0.0 0.0"/>
                 </external_part>
-                <!-- <internal_part name="Foam" type="cylinder" physics="surface" buoyant="true">
-                    <dimensions radius="0.2" height="0.9"/>
-                    <origin rpy="0.0 0.0 0.0" xyz="0.0 0.0 -0.5"/>
-                    <material name="Foam"/>
-                    <mass value="0.0"/>
-                    <look name="grey"/>
-                    <compound_transform rpy="0.0 0 0.0" xyz="0 0.0 0"/>
-                </internal_part> -->
+                <external_part name="engine_starboard" type="model" physics="submerged" bouyant="true">
+                    <physical>
+                        <mesh filename="engine.obj" scale="0.5"/>
+                        <origin rpy="3.14 0 0" xyz="-1 .45 -.2"/>
+                    </physical>
+                    <visual>
+                        <mesh filename="engine.obj" scale="0.5"/>
+                        <origin rpy="3.14 0 0" xyz="-1 .45 -.2"/>
+                    </visual>
+                    <material name="Vehicle"/>
+                    <look name="yellow"/>
+                    <mass value="10"/>
+                    <compound_transform rpy="0.0 0.0 0.0" xyz="0.0 0.0 0.0"/>
+                    <cg xyz=" 0.0 0 1.0" rpy="0.0 0.0 0.0"/>
+                </external_part>
+                <external_part name="engine_port" type="model" physics="submerged" bouyant="true">
+                    <physical>
+                        <mesh filename="engine.obj" scale="0.5"/>
+                        <origin rpy="3.14 0 0" xyz="-1 -.45 -.2"/>
+                    </physical>
+                    <visual>
+                        <mesh filename="engine.obj" scale="0.5"/>
+                        <origin rpy="3.14 0 0" xyz="-1 -.45 -.2"/>
+                    </visual>
+                    <material name="Vehicle"/>
+                    <look name="yellow"/>
+                    <mass value="10"/>
+                    <compound_transform rpy="0.0 0.0 0.0" xyz="0.0 0.0 0.0"/>
+                    <cg xyz=" 0.0 0 1.0" rpy="0.0 0.0 0.0"/>
+                </external_part>
             </base_link>
             <!-- the actual base frame  -->

File: wamv_stonefish/scenarios/tank.scn.xacro (robot description, xacro)
@@ -9,5 +9,5 @@
 <scenario xmlns:xacro="http://ros.org/wiki/xacro">
     <xacro:arg name="robot_name" default="changeme"/>
-    <xacro:include filename="$(find alpha_std_stonefish)/description/alpha_std.scn.xacro"/>
+    <xacro:include filename="$(find wamv_stonefish)/description/wamv.scn.xacro"/>
     <xacro:alpha_sci robot_name="$(arg robot_name)" xyz="0.0 0.0 0.0" rpy="0.0 0.0 0.0"/>
     <environment>

Commit message: feat:props and keyboard teleop

File: wamv_stonefish/description/wamv.scn.xacro (robot description, xacro)
@@ -58,4 +58,30 @@
                     <cg xyz=" 0.0 0 1.0" rpy="0.0 0.0 0.0"/>
                 </external_part>
+                <external_part name="thrusterPort" type="model" physics="submerged" buoyant="false">
+                    <physical>
+                        <mesh filename="propeller.obj" scale="0.5"/>
+                        <origin rpy="0.0 0 0.0" xyz="-1.1 -.45 0.08"/>
+                    </physical>
+                    <visual>
+                        <mesh filename="propeller.obj" scale="0.5"/>
+                        <origin rpy="0.0 0 0.0" xyz="-1.1 -.45 0.08"/>
+                    </visual>
+                    <material name="Neutral"/>
+                    <look name="black"/>
+                    <compound_transform rpy="0.0 0.0 0.0" xyz="0.0 0.0 0.0"/>
+                </external_part>
+                <external_part name="thrusterStarboard" type="model" physics="submerged" buoyant="false">
+                    <physical>
+                        <mesh filename="propeller.obj" scale="0.5"/>
+                        <origin rpy="0.0 0 0.0" xyz="-1.1 .45 0.08"/>
+                    </physical>
+                    <visual>
+                        <mesh filename="propeller.obj" scale="0.5"/>
+                        <origin rpy="0.0 0 0.0" xyz="-1.1 .45 0.08"/>
+                    </visual>
+                    <material name="Neutral"/>
+                    <look name="black"/>
+                    <compound_transform rpy="0.0 0.0 0.0" xyz="0.0 0.0 0.0"/>
+                </external_part>
             </base_link>
             <!-- the actual base frame  -->
@@ -72,4 +98,26 @@
                 <axis xyz="1.0 0.0 0.0"/>
             </joint>
+            <actuator name="ThrusterPort" type="thruster">
+                <link name="Base"/>
+                <origin rpy="0.0 0.0 0" xyz="-1.1 -.45 0.08"/>
+                <specs thrust_coeff="0.4315" thrust_coeff_backward="0.3404" torque_coeff="0.01" max_rpm="3000.0"/>
+                <propeller diameter="0.08" right="true">
+                    <mesh filename="propeller.obj" scale="0.5"/>
+                    <material name="Neutral"/>
+                    <look name="white"/>
+                </propeller>
+                <ros_subscriber topic="/${robot_name}/control/thruster/port"/>
+            </actuator>
+            <actuator name="ThrusterStarboard" type="thruster">
+                <link name="Base"/>
+                <origin rpy="0.0 0.0 0" xyz="-1.1 .45 0.08"/>
+                <specs thrust_coeff="0.4315" thrust_coeff_backward="0.3404" torque_coeff="0.01" max_rpm="3000.0"/>
+                <propeller diameter="0.08" right="true">
+                    <mesh filename="propeller.obj" scale="0.5"/>
+                    <material name="Neutral"/>
+                    <look name="white"/>
+                </propeller>
+                <ros_subscriber topic="/${robot_name}/control/thruster/starboard"/>
+            </actuator>
             <world_transform rpy="${rpy}" xyz="${xyz}"/>
         </robot>

Commit message: feat: Added a camera

File: wamv_stonefish/description/wamv.scn.xacro (robot description, xacro)
@@ -198,4 +198,10 @@
                 <link name="Base"/>
             </sensor>
+            <sensor name="Cam" rate="10.0" type="camera">
+                <specs resolution_x="800" resolution_y="600" horizontal_fov="60.0"/>
+                <origin xyz="0.0 0.0 -0.3" rpy="-1.57 3.14 4.71"/>
+                <link name="Base"/>
+                <ros_publisher topic="/${robot_name}/camera/stonefish/data"/>
+            </sensor>
             <world_transform rpy="${rpy}" xyz="${xyz}"/>
         </robot>
