Commit message: feat:multibeam added

File: wamv_description/urdf/base.urdf.xacro (robot description, xacro)
@@ -15,3 +15,9 @@
         <child link="cg_link"/>
     </joint>
+    <link name="Multibeam"/>
+    <joint name="Multibeam_joint" type="fixed">
+        <origin xyz="0.0 0.0 0.0" rpy="1.57 0.0 1.57"/>
+        <parent link="base_link"/>
+        <child link="Multibeam"/>
+    </joint>
 </robot>

File: wamv_stonefish/description/wamv.scn.xacro (robot description, xacro)
@@ -120,4 +120,13 @@
                 <ros_subscriber topic="/${robot_name}/control/thruster/starboard"/>
             </actuator>
+            <sensor name="Multibeam" rate="10" type="multibeam">
+                <specs fov="120.0" steps="128"/>
+                <range distance_min="0.5" distance_max="50.0"/>
+                <noise distance="0.1"/>
+                <history samples="1"/>
+                <origin xyz="0.0 0.0 .1" rpy="1.57 0.0 1.57"/>
+                <link name="Vehicle"/>
+                <ros_publisher topic="/${robot_name}/multibeam_sonar/stonefish/data"/>
+            </sensor>
             <world_transform rpy="${rpy}" xyz="${xyz}"/>
         </robot>

Commit message: fix:tf btwn base and sonar

File: wamv_description/urdf/base.urdf.xacro (robot description, xacro)
@@ -1,4 +1,5 @@
 <?xml version="1.0"?>
 <robot name="alpha_std" xmlns:xacro="http://ros.org/wiki/xacro">
+    <!--This operates in std frame-->
     <link name="base_link">
         <visual>
@@ -17,5 +18,5 @@
     <link name="Multibeam"/>
     <joint name="Multibeam_joint" type="fixed">
-        <origin xyz="0.0 0.0 0.0" rpy="1.57 0.0 1.57"/>
+        <origin xyz="0.0 0.0 -0.1" rpy="-1.57 .785 0"/>
         <parent link="base_link"/>
         <child link="Multibeam"/>

File: wamv_stonefish/description/wamv.scn.xacro (robot description, xacro)
@@ -6,4 +6,5 @@
     Year: 2023
     Copyright (C) 2022 Smart Ocean Systems Laboratory
+    This file operates in NED Frame
 -->
 <scenario xmlns:xacro="http://ros.org/wiki/xacro">
@@ -121,9 +122,9 @@
             </actuator>
             <sensor name="Multibeam" rate="10" type="multibeam">
-                <specs fov="120.0" steps="128"/>
-                <range distance_min="0.5" distance_max="50.0"/>
+                <specs fov="90.0" steps="256"/>
+                <range distance_min="0.5" distance_max="100.0"/>
                 <noise distance="0.1"/>
                 <history samples="1"/>
-                <origin xyz="0.0 0.0 .1" rpy="1.57 0.0 1.57"/>
+                <origin xyz="0.0 0.0 .1" rpy="1.57 -.785 1.57"/>
                 <link name="Vehicle"/>
                 <ros_publisher topic="/${robot_name}/multibeam_sonar/stonefish/data"/>

File: wamv_stonefish/scenarios/ocean.scn.xacro (robot description, xacro)
@@ -41,5 +41,5 @@
         <material name="Rock"/>
         <look name="Gray"/>
-        <world_transform xyz="0.0 0.0 40.0" rpy="0.0 0.0 0.0"/>
+        <world_transform xyz="0.0 0.0 60.0" rpy="0.0 0.0 0.0"/>
     </static>
 </scenario>

Commit message: feat:added imu+gps

File: wamv_description/urdf/base.urdf.xacro (robot description, xacro)
@@ -16,9 +16,21 @@
         <child link="cg_link"/>
     </joint>
-    <link name="Multibeam"/>
-    <joint name="Multibeam_joint" type="fixed">
-        <origin xyz="0.0 0.0 -0.1" rpy="-1.57 .785 0"/>
+    <link name="multibeam"/>
+    <joint name="multibeam_joint" type="fixed">
+        <origin xyz="0.0 0.0 -0.1" rpy="-1.57 .785 -1.57"/>
         <parent link="base_link"/>
-        <child link="Multibeam"/>
+        <child link="multibeam"/>
+    </joint>
+    <link name="imu_sf"/>
+    <joint name="imu__sf_joint" type="fixed">
+        <origin xyz="0.0 0.0 0.0" rpy="0.0 0.0 0.0"/>
+        <parent link="base_link"/>
+        <child link="imu_sf"/>
+    </joint>
+    <link name="gps"/>
+    <joint name="gps_joint" type="fixed">
+        <origin xyz="0.0 0.0 0.28" rpy="3.1415926 0.0 -1.5707963"/>
+        <parent link="base_link"/>
+        <child link="gps"/>
     </joint>
 </robot>

File: wamv_stonefish/description/wamv.scn.xacro (robot description, xacro)
@@ -121,5 +121,5 @@
                 <ros_subscriber topic="/${robot_name}/control/thruster/starboard"/>
             </actuator>
-            <sensor name="Multibeam" rate="10" type="multibeam">
+            <sensor name="multibeam" rate="10" type="multibeam">
                 <specs fov="90.0" steps="256"/>
                 <range distance_min="0.5" distance_max="100.0"/>
@@ -127,6 +127,18 @@
                 <history samples="1"/>
                 <origin xyz="0.0 0.0 .1" rpy="1.57 -.785 1.57"/>
-                <link name="Vehicle"/>
+                <link name="Base"/>
                 <ros_publisher topic="/${robot_name}/multibeam_sonar/stonefish/data"/>
+            </sensor>
+            <sensor name="imu_sf" type="imu" rate="20.0">
+                <link name="Base"/>
+                <origin rpy="3.1415926 0.0 0.0" xyz="0 0.0 -0.05"/>
+                <noise angle="0.01 0.01 0.05" angular_velocity="0.05" yaw_drift="0.001" linear_acceleration="0.1"/>
+                <ros_publisher topic="/${robot_name}/imu/stonefish/data"/>
+            </sensor>
+            <sensor name="gps" type="gps" rate="1.0">
+                <link name="Base"/>
+                <origin rpy="0.0 0.0 0.0" xyz="-0.7 0.0 -0.3"/>
+                <noise ned_position="0.1"/>
+                <ros_publisher topic="/${robot_name}/gps/fix"/>
             </sensor>
             <world_transform rpy="${rpy}" xyz="${xyz}"/>

Commit message: fix:tf btwn odom and multibeam

File: wamv_description/urdf/base.urdf.xacro (robot description, xacro)
@@ -22,9 +22,9 @@
         <child link="multibeam"/>
     </joint>
-    <link name="imu_sf"/>
+    <link name="imu"/>
     <joint name="imu__sf_joint" type="fixed">
         <origin xyz="0.0 0.0 0.0" rpy="0.0 0.0 0.0"/>
         <parent link="base_link"/>
-        <child link="imu_sf"/>
+        <child link="imu"/>
     </joint>
     <link name="gps"/>

File: wamv_stonefish/description/wamv.scn.xacro (robot description, xacro)
@@ -130,5 +130,5 @@
                 <ros_publisher topic="/${robot_name}/multibeam_sonar/stonefish/data"/>
             </sensor>
-            <sensor name="imu_sf" type="imu" rate="20.0">
+            <sensor name="imu" type="imu" rate="20.0">
                 <link name="Base"/>
                 <origin rpy="3.1415926 0.0 0.0" xyz="0 0.0 -0.05"/>

Commit message: ft: lidar tf

File: wamv_description/urdf/base.urdf.xacro (robot description, xacro)
@@ -22,4 +22,16 @@
         <child link="multibeam"/>
     </joint>
+    <!-- <link name="laserscanner_1"/>
+    <joint name="laserscanner_1_joint" type="fixed">
+        <origin xyz="0.0 0.0 1" rpy="-0 0 0"/>
+        <parent link="base_link"/>
+        <child link="laserscanner_1"/>
+    </joint> -->
+    <link name="laserscanner_2"/>
+    <joint name="laserscanner_2_joint" type="fixed">
+        <origin xyz="0.0 0.0 5" rpy="0 0 4.712389"/>
+        <parent link="base_link"/>
+        <child link="laserscanner_2"/>
+    </joint>
     <link name="imu"/>
     <joint name="imu__sf_joint" type="fixed">

File: wamv_stonefish/description/wamv.scn.xacro (robot description, xacro)
@@ -130,8 +130,28 @@
                 <ros_publisher topic="/${robot_name}/multibeam_sonar/stonefish/data"/>
             </sensor>
+            <!-- <sensor name="laserscanner_1" rate="10" type="multibeam">
+                <specs fov="45" steps="128"/>
+                <range distance_min="0.5" distance_max="100.0"/>
+                <noise distance="0.1"/>
+                <history samples="1"/>
+                <origin xyz="0.0 0.0 -1" rpy="0 0 1.57"/>
+                <link name="Base"/>
+                <ros_publisher topic="/${robot_name}/laserscanner_1/stonefish/data"/>
+            </sensor> -->
+            <sensor name="laserscanner_2" rate="10" type="multibeam">
+                <specs fov="45" steps="128"/>
+                <range distance_min="0.5" distance_max="100.0"/>
+                <!-- <noise distance="0.1"/> -->
+                <noise distance="0.0"/>
+                <history samples="1"/>
+                <origin xyz="0.0 0.0 -5" rpy="3.14 0 -4.712389"/>
+                <link name="Base"/>
+                <ros_publisher topic="/${robot_name}/laserscanner_2/stonefish/data"/>
+            </sensor>
             <sensor name="imu" type="imu" rate="20.0">
                 <link name="Base"/>
                 <origin rpy="3.1415926 0.0 0.0" xyz="0 0.0 -0.05"/>
-                <noise angle="0.01 0.01 0.05" angular_velocity="0.05" yaw_drift="0.001" linear_acceleration="0.1"/>
+                <!-- <noise angle="0.01 0.01 0.05" angular_velocity="0.05" yaw_drift="0.001" linear_acceleration="0.1"/> -->
+                <noise angle="0.0 0.0 0.0" angular_velocity="0.0" yaw_drift="0.00" linear_acceleration="0.0"/>
                 <ros_publisher topic="/${robot_name}/imu/stonefish/data"/>
             </sensor>
@@ -139,5 +159,6 @@
                 <link name="Base"/>
                 <origin rpy="0.0 0.0 0.0" xyz="-0.7 0.0 -0.3"/>
-                <noise ned_position="0.1"/>
+                <!-- <noise ned_position="0.1"/> -->
+                <noise ned_position="0.0"/>
                 <ros_publisher topic="/${robot_name}/gps/fix"/>
             </sensor>

Commit message: feat: Lidar implemented at 0 localisation noise

File: wamv_description/urdf/base.urdf.xacro (robot description, xacro)
@@ -22,15 +22,33 @@
         <child link="multibeam"/>
     </joint>
-    <!-- <link name="laserscanner_1"/>
+    <link name="laserscanner_1"/>
     <joint name="laserscanner_1_joint" type="fixed">
-        <origin xyz="0.0 0.0 1" rpy="-0 0 0"/>
+        <origin xyz="0.0 0.0 0.1" rpy="0 -0.0 4.712389"/>
         <parent link="base_link"/>
         <child link="laserscanner_1"/>
-    </joint> -->
-    <link name="laserscanner_2"/>
-    <joint name="laserscanner_2_joint" type="fixed">
-        <origin xyz="0.0 0.0 5" rpy="0 0 4.712389"/>
+    </joint>
+    <link name="laserscanner_3"/>
+    <joint name="laserscanner_3_joint" type="fixed">
+        <origin xyz="0.0 0.0 0.1" rpy="0 -0.08726646 4.712389"/>
         <parent link="base_link"/>
-        <child link="laserscanner_2"/>
+        <child link="laserscanner_3"/>
+    </joint>
+    <link name="laserscanner_5"/>
+    <joint name="laserscanner_5_joint" type="fixed">
+        <origin xyz="0.0 0.0 0.1" rpy="0 -0.1745329 4.712389"/>
+        <parent link="base_link"/>
+        <child link="laserscanner_5"/>
+    </joint>
+    <link name="laserscanner_7"/>
+    <joint name="laserscanner_7_joint" type="fixed">
+        <origin xyz="0.0 0.0 0.1" rpy="0 -0.2617994 4.712389"/>
+        <parent link="base_link"/>
+        <child link="laserscanner_7"/>
+    </joint>
+    <link name="laserscanner_9"/>
+    <joint name="laserscanner_9_joint" type="fixed">
+        <origin xyz="0.0 0.0 0.1" rpy="0 -0.3490659 4.712389"/>
+        <parent link="base_link"/>
+        <child link="laserscanner_9"/>
     </joint>
     <link name="imu"/>

File: wamv_stonefish/description/wamv.scn.xacro (robot description, xacro)
@@ -130,22 +130,48 @@
                 <ros_publisher topic="/${robot_name}/multibeam_sonar/stonefish/data"/>
             </sensor>
-            <!-- <sensor name="laserscanner_1" rate="10" type="multibeam">
-                <specs fov="45" steps="128"/>
+            <sensor name="laserscanner_1" rate="10" type="multibeam">
+                <specs fov="45" steps="64"/>
                 <range distance_min="0.5" distance_max="100.0"/>
                 <noise distance="0.1"/>
                 <history samples="1"/>
-                <origin xyz="0.0 0.0 -1" rpy="0 0 1.57"/>
+                <origin xyz="0.0 0.0 -0.6" rpy="3.14 0 -4.712389"/>
                 <link name="Base"/>
                 <ros_publisher topic="/${robot_name}/laserscanner_1/stonefish/data"/>
-            </sensor> -->
-            <sensor name="laserscanner_2" rate="10" type="multibeam">
-                <specs fov="45" steps="128"/>
+            </sensor>
+            <sensor name="laserscanner_3" rate="10" type="multibeam">
+                <specs fov="45" steps="64"/>
                 <range distance_min="0.5" distance_max="100.0"/>
-                <!-- <noise distance="0.1"/> -->
-                <noise distance="0.0"/>
+                <noise distance="0.1"/>
                 <history samples="1"/>
-                <origin xyz="0.0 0.0 -5" rpy="3.14 0 -4.712389"/>
+                <origin xyz="0.0 0.0 -0.6" rpy="3.14 0.08726646 -4.712389"/>
                 <link name="Base"/>
-                <ros_publisher topic="/${robot_name}/laserscanner_2/stonefish/data"/>
+                <ros_publisher topic="/${robot_name}/laserscanner_3/stonefish/data"/>
+            </sensor>
+            <sensor name="laserscanner_5" rate="1" type="multibeam">
+                <specs fov="45" steps="64"/>
+                <range distance_min="0.5" distance_max="100.0"/>
+                <noise distance="0.1"/>
+                <history samples="1"/>
+                <origin xyz="0.0 0.0 -0.6" rpy="3.14 0.1745329 -4.712389"/>
+                <link name="Base"/>
+                <ros_publisher topic="/${robot_name}/laserscanner_5/stonefish/data"/>
+            </sensor>
+            <sensor name="laserscanner_7" rate="1" type="multibeam">
+                <specs fov="45" steps="64"/>
+                <range distance_min="0.5" distance_max="100.0"/>
+                <noise distance="0.1"/>
+                <history samples="1"/>
+                <origin xyz="0.0 0.0 -0.6" rpy="3.14 0.2617994 -4.712389"/>
+                <link name="Base"/>
+                <ros_publisher topic="/${robot_name}/laserscanner_7/stonefish/data"/>
+            </sensor>
+            <sensor name="laserscanner_9" rate="1" type="multibeam">
+                <specs fov="45" steps="64"/>
+                <range distance_min="0.5" distance_max="100.0"/>
+                <noise distance="0.1"/>
+                <history samples="1"/>
+                <origin xyz="0.0 0.0 -0.6" rpy="3.14 0.3490659 -4.712389"/>
+                <link name="Base"/>
+                <ros_publisher topic="/${robot_name}/laserscanner_9/stonefish/data"/>
             </sensor>
             <sensor name="imu" type="imu" rate="20.0">

Commit message: feat: msis

File: wamv_description/urdf/base.urdf.xacro (robot description, xacro)
@@ -64,3 +64,9 @@
         <child link="gps"/>
     </joint>
+    <link name="msis"/>
+    <joint name="msis_joint" type="fixed">
+        <origin xyz="0.0 0.0 0.1" rpy="0 0 0"/>
+        <parent link="base_link"/>
+        <child link="msis"/>
+    </joint>
 </robot>

File: wamv_stonefish/description/wamv.scn.xacro (robot description, xacro)
@@ -189,4 +189,13 @@
                 <ros_publisher topic="/${robot_name}/gps/fix"/>
             </sensor>
+            <sensor name="MSIS" type="msis">
+                <specs step="0.25" bins="500" horizontal_beam_width="2.0" vertical_beam_width="30.0"/>
+                <settings range_min="0.5" range_max="10.0" rotation_min="-50.0" rotation_max="50.0" gain="1.5"/>
+                <noise multiplicative="0.02" additive="0.03"/>
+                <display colormap="hot"/>
+                <origin xyz="0.0 0.0 0.0" rpy="-1.57 3.14 4.71"/>
+                <ros_publisher topic="/${robot_name}/msis/stonefish/data"/>
+                <link name="Base"/>
+            </sensor>
             <world_transform rpy="${rpy}" xyz="${xyz}"/>
         </robot>

Commit message: added:tf for thrusters

File: wamv_description/urdf/base.urdf.xacro (robot description, xacro)
@@ -6,5 +6,5 @@
             <origin xyz="0.0 -0 -0" rpy="0.0 0.0 0"/>
             <geometry>
-                <mesh filename="package://wamv_description/mesh/wamv_base.obj" scale="0.001 0.001 0.001"/>
+                <mesh filename="package://wamv_description/mesh/wamv_base.obj" scale="0.0045 0.0045 0.0045"/>
             </geometry>
         </visual>
@@ -18,5 +18,5 @@
     <link name="multibeam"/>
     <joint name="multibeam_joint" type="fixed">
-        <origin xyz="0.0 0.0 -0.1" rpy="-1.57 .785 -1.57"/>
+        <origin xyz="0.0 0.0 -0.5" rpy="-1.57 .785 -1.57"/>
         <parent link="base_link"/>
         <child link="multibeam"/>
@@ -24,5 +24,5 @@
     <link name="laserscanner_1"/>
     <joint name="laserscanner_1_joint" type="fixed">
-        <origin xyz="0.0 0.0 0.1" rpy="0 -0.0 4.712389"/>
+        <origin xyz="0.0 0.0 0.5" rpy="0 -0.0 4.712389"/>
         <parent link="base_link"/>
         <child link="laserscanner_1"/>
@@ -30,5 +30,5 @@
     <link name="laserscanner_3"/>
     <joint name="laserscanner_3_joint" type="fixed">
-        <origin xyz="0.0 0.0 0.1" rpy="0 -0.08726646 4.712389"/>
+        <origin xyz="0.0 0.0 0.5" rpy="0 -0.08726646 4.712389"/>
         <parent link="base_link"/>
         <child link="laserscanner_3"/>
@@ -36,5 +36,5 @@
     <link name="laserscanner_5"/>
     <joint name="laserscanner_5_joint" type="fixed">
-        <origin xyz="0.0 0.0 0.1" rpy="0 -0.1745329 4.712389"/>
+        <origin xyz="0.0 0.0 0.5" rpy="0 -0.1745329 4.712389"/>
         <parent link="base_link"/>
         <child link="laserscanner_5"/>
@@ -42,5 +42,5 @@
     <link name="laserscanner_7"/>
     <joint name="laserscanner_7_joint" type="fixed">
-        <origin xyz="0.0 0.0 0.1" rpy="0 -0.2617994 4.712389"/>
+        <origin xyz="0.0 0.0 0.5" rpy="0 -0.2617994 4.712389"/>
         <parent link="base_link"/>
         <child link="laserscanner_7"/>
@@ -48,5 +48,5 @@
     <link name="laserscanner_9"/>
     <joint name="laserscanner_9_joint" type="fixed">
-        <origin xyz="0.0 0.0 0.1" rpy="0 -0.3490659 4.712389"/>
+        <origin xyz="0.0 0.0 0.5" rpy="0 -0.3490659 4.712389"/>
         <parent link="base_link"/>
         <child link="laserscanner_9"/>
@@ -66,7 +66,19 @@
     <link name="msis"/>
     <joint name="msis_joint" type="fixed">
-        <origin xyz="0.0 0.0 0.1" rpy="0 0 0"/>
+        <origin xyz="0.0 0.0 0.5" rpy="0 0 0"/>
         <parent link="base_link"/>
         <child link="msis"/>
     </joint>
+    <link name="thruster_starboard_link"/>
+    <joint name="thruster_starboard_joint" type="fixed">
+        <origin rpy="0 0 0" xyz="-1 -.45 -.2"/>
+        <parent link="base_link"/>
+        <child link="thruster_starboard_link"/>
+    </joint>
+    <link name="thruster_port_link"/>
+    <joint name="thruster_port_joint" type="fixed">
+        <origin rpy="0 0 0" xyz="-1 .45 -.2"/>
+        <parent link="base_link"/>
+        <child link="thruster_port_link"/>
+    </joint>
 </robot>

Commit message: fix: removed msis from wamv

File: wamv_description/urdf/base.urdf.xacro (robot description, xacro)
@@ -64,4 +64,5 @@
         <child link="gps"/>
     </joint>
+<!--
     <link name="msis"/>
     <joint name="msis_joint" type="fixed">
@@ -69,8 +70,8 @@
         <parent link="base_link"/>
         <child link="msis"/>
-    </joint>
+    </joint> -->
     <link name="thruster_starboard_link"/>
     <joint name="thruster_starboard_joint" type="fixed">
-        <origin rpy="0 0 0" xyz="-1 -.45 -.2"/>
+        <origin rpy="3.14 0 0" xyz="-1 -.45 -.2"/>
         <parent link="base_link"/>
         <child link="thruster_starboard_link"/>
@@ -78,5 +79,5 @@
     <link name="thruster_port_link"/>
     <joint name="thruster_port_joint" type="fixed">
-        <origin rpy="0 0 0" xyz="-1 .45 -.2"/>
+        <origin rpy="3.14 0 0" xyz="-1 .45 -.2"/>
         <parent link="base_link"/>
         <child link="thruster_port_link"/>

Commit message: updated path_global (prev.) refs to path_3d (current)

File: wamv_description/urdf/base.urdf.xacro (robot description, xacro)
@@ -64,4 +64,10 @@
         <child link="gps"/>
     </joint>
+    <link name="USBL"/>
+    <joint name="USBL_joint" type="fixed">
+        <origin xyz="0.0 0.0 0.0" rpy="0.0 0.0 0.0"/>
+        <parent link="base_link"/>
+        <child link="USBL"/>
+    </joint>
 <!--
     <link name="msis"/>

Commit message: temporary branch to fix localization issue

File: wamv_description/urdf/base.urdf.xacro (robot description, xacro)
@@ -22,5 +22,5 @@
         <child link="multibeam"/>
     </joint>
-    <link name="laserscanner_1"/>
+    <!-- <link name="laserscanner_1"/>
     <joint name="laserscanner_1_joint" type="fixed">
         <origin xyz="0.0 0.0 0.5" rpy="0 -0.0 4.712389"/>
@@ -51,22 +51,41 @@
         <parent link="base_link"/>
         <child link="laserscanner_9"/>
-    </joint>
+    </joint> -->
     <link name="imu"/>
-    <joint name="imu__sf_joint" type="fixed">
+    <joint name="imu_joint" type="fixed">
         <origin xyz="0.0 0.0 0.0" rpy="0.0 0.0 0.0"/>
         <parent link="base_link"/>
         <child link="imu"/>
     </joint>
+    <link name="imu_sf"/>
+    <joint name="imu_sf_joint" type="fixed">
+        <origin xyz="0.0 0.0 0.0" rpy="0.0 0.0 0.0"/>
+        <parent link="base_link"/>
+        <child link="imu_sf"/>
+    </joint>
     <link name="gps"/>
     <joint name="gps_joint" type="fixed">
-        <origin xyz="0.0 0.0 0.28" rpy="3.1415926 0.0 -1.5707963"/>
+        <origin xyz="-0.7 0.0 0.3" rpy="3.1415926 0.0 0.0"/>
         <parent link="base_link"/>
         <child link="gps"/>
     </joint>
-    <link name="USBL"/>
-    <joint name="USBL_joint" type="fixed">
-        <origin xyz="0.0 0.0 0.0" rpy="0.0 0.0 0.0"/>
+    <link name="dvl_sf"/>
+    <joint name="dvl_sf_joint" type="fixed">
+        <origin xyz="-0.65 0.0 0.1" rpy="0.0 0.0 0.0"/>
         <parent link="base_link"/>
-        <child link="USBL"/>
+        <child link="dvl_sf"/>
+    </joint>
+    <link name="usbl"/>
+    <joint name="usbl_joint" type="fixed">
+        <origin xyz="-0.1 0.0 -0.5" rpy="0.0 3.1415926 3.1415926"/>
+        <parent link="base_link"/>
+        <child link="usbl"/>
+    </joint>
+    <link name="HydromeaUVX"/>
+    <joint name="HydromeaUVX_joint" type="fixed">
+        <origin xyz="0.0 0.0 -0.5" rpy="3.6652 0.0 0.0"/>
+        <!-- <origin xyz="0.0 0.0 -0.5" rpy="4.18879 0.0 0.0"/> -->
+        <parent link="base_link"/>
+        <child link="HydromeaUVX"/>
     </joint>
 <!--
