Commit message: added a single multibeam to emulate some VLP16 LiDAR data. todo: add more multibeams to emulate more channels

File: wamv_description/urdf/base.urdf.xacro (robot description, xacro)
@@ -22,5 +22,5 @@
         <child link="multibeam"/>
     </joint>
-    <!-- <link name="laserscanner_1"/>
+    <link name="laserscanner_1"/>
     <joint name="laserscanner_1_joint" type="fixed">
         <origin xyz="0.0 0.0 0.5" rpy="0 -0.0 4.712389"/>
@@ -51,5 +51,11 @@
         <parent link="base_link"/>
         <child link="laserscanner_9"/>
-    </joint> -->
+    </joint>
+    <link name="vlp16"/>
+    <joint name="vlp16_joint" type="fixed">
+        <origin xyz="0.00 0.00 1.0" rpy="3.14159 0.00 0.00"/>
+        <parent link="base_link"/>
+        <child link="vlp16"/>
+    </joint>
     <link name="imu"/>
     <joint name="imu_joint" type="fixed">
@@ -66,5 +72,5 @@
     <link name="gps"/>
     <joint name="gps_joint" type="fixed">
-        <origin xyz="-0.7 0.0 0.3" rpy="3.1415926 0.0 0.0"/>
+        <origin xyz="0.0 0.0 0.3" rpy="3.1415926 0.0 0.0"/>
         <parent link="base_link"/>
         <child link="gps"/>

Commit message: optical modem joint + PID updates

File: wamv_description/urdf/base.urdf.xacro (robot description, xacro)
@@ -90,6 +90,7 @@
     <link name="HydromeaUVX"/>
     <joint name="HydromeaUVX_joint" type="fixed">
-        <origin xyz="0.0 0.0 -0.5" rpy="3.6652 0.0 0.0"/>
-        <!-- <origin xyz="0.0 0.0 -0.5" rpy="4.18879 0.0 0.0"/> -->
+        <origin xyz="0.0 0.0 -0.5" rpy="1.5708 2.0944 1.5708"/>
+        <!-- <origin xyz="0.0 0.0 -0.5" rpy="3.6652 0.0 0.0"/> -->
+        <!-- <origin xyz="0.0 0.0 -0.5" rpy="3.1415926 0.0 0.0"/> -->
         <parent link="base_link"/>
         <child link="HydromeaUVX"/>
